Commit message: feat: add wheel system and joint state publishing to robot model
- Add left, right, and caster wheel links and joints in URDF
- Connect all wheel links to base_link via proper joints
- Integrate joint_state_publisher for TF generation and RViz visualization

docs: update NOTES.md to reflect URDF and launch file changes

File: src/rover_description/urdf/rover.urdf (robot description, URDF)
Before this commit: robot rover_bot, 2 links, 1 joints
Links:
- removed link dummy_link
- added link caster_wheel; visual sphere radius=0.05
- added link left_wheel; visual cylinder length=0.02 radius=0.07
- added link right_wheel; visual cylinder length=0.02 radius=0.07
Joints:
- removed joint base_to_dummy
- added joint caster_joint: type fixed, parent base_link, child caster_wheel, origin xyz=-0.2 0 0.05
- added joint left_wheel_joint: type continuous, parent base_link, child left_wheel, origin xyz=0.2 0.16 0.07 rpy=1.57 1.57 0, axis 0 0 1
- added joint right_wheel_joint: type continuous, parent base_link, child right_wheel, origin xyz=0.2 -0.16 0.07 rpy=1.57 1.57 0, axis 0 0 1

Commit message: feat: restructure robot model, add Gazebo simulation, and RViz config
- refactor URDF: introduce chassis link and use it in joints; base_link is now an empty root link
- add collision and inertial tags to improve physical simulation
- add RViz configuration file and update display launch file to load it
- create rover_gazebo package for simulation
- add empty.sdf world file for Gazebo
- add launch file to start Gazebo and spawn rover_bot
- update NOTES.md with structured project-specific sections reflecting recent changes

File: src/rover_description/urdf/rover.urdf (robot description, URDF)
Before this commit: robot rover_bot, 4 links, 3 joints
Links:
- added link chassis, mass 5.0; collision box size=0.5 0.3 0.1; visual box size=0.5 0.3 0.1
- link base_link: geometry 
- link caster_wheel: mass None -> 0.2; geometry collision sphere radius=0.05; visual sphere radius=0.05
- link left_wheel: mass None -> 0.5; geometry collision cylinder length=0.02 radius=0.07; visual cylinder length=0.02 radius=0.07
- link right_wheel: mass None -> 0.5; geometry collision cylinder length=0.02 radius=0.07; visual cylinder length=0.02 radius=0.07
Joints:
- added joint base_to_chassis: type fixed, parent base_link, child chassis, origin xyz= -0.1 0 0
- joint caster_joint: parent base_link -> chassis
- joint left_wheel_joint: origin xyz=0.2 0.16 0.07 rpy=1.57 1.57 0 -> xyz=0.2 0.16 0.07 rpy=-1.57 0 0; parent base_link -> chassis
- joint right_wheel_joint: axis 0 0 1 -> 0 0 -1; origin xyz=0.2 -0.16 0.07 rpy=1.57 1.57 0 -> xyz=0.2 -0.16 0.07 rpy=1.57 0 0; parent base_link -> chassis

Commit message: feat(simulation): integrate LiDAR and update Gazebo world and launch setup
- extend URDF with LiDAR link and Gazebo sensor configuration
- add topic bridges for drive commands and LiDAR data
- fix robot_description parameter handling using ParameterValue(str) to prevent YAML parsing/SDF issues
- overhaul world file (empty.sdf):
  - remove external Fuel assets
  - define local ground plane and lighting
  - include necessary simulation plugins

File: src/rover_description/urdf/rover.urdf (robot description, URDF)
Before this commit: robot rover_bot, 5 links, 4 joints
Links:
- added link lidar_link, mass 0.1; collision cylinder length=0.02 radius=0.05; visual cylinder length=0.02 radius=0.05
Joints:
- added joint lidar_joint: type fixed, parent chassis, child lidar_link, origin xyz=0.2 0 0.15

Commit message: feat(simulation): improve URDF, launch, and Gazebo setup
- Add `gz_frame_id` to sensor tag in URDF to fix "queue full" issue when RViz displays LiDAR via LaserScan.
- Create `config/bridge.yaml` to simplify launch files and consolidate bridge node configuration.
- Add bridge config file path in `setup.py`.
- Add `-r` flag to Gazebo execute process in launch file for direct simulation start.
- Enable `use_sim_time` for all relevant nodes in launch file.
- Export current Gazebo world to `world_07-05-2026`.

File: src/rover_description/urdf/rover.urdf (robot description, URDF)
Before this commit: robot rover_bot, 6 links, 5 joints
Links:
- removed link chassis
- added link base_footprint
- link base_link: mass None -> 5.0; geometry collision box size=0.5 0.3 0.1; visual box size=0.5 0.3 0.1
Joints:
- removed joint base_to_chassis
- added joint base_to_base_link: type fixed, parent base_footprint, child base_link, origin xyz= -0.1 0 0
- joint caster_joint: parent chassis -> base_link
- joint left_wheel_joint: parent chassis -> base_link
- joint lidar_joint: parent chassis -> base_link
- joint right_wheel_joint: parent chassis -> base_link

Commit message: fix(urdf): improve wheel-ground interaction and stabilize rotation in simulation
- Add damping and friction to wheel joints for smoother dynamics
- Add mu1 and mu2 parameters to wheel contact surfaces
- Fix unstable rotation behavior in Gazebo simulation

File: src/rover_description/urdf/rover.urdf (robot description, URDF)
Before this commit: robot rover_bot, 6 links, 5 joints
Joints:
- joint base_to_base_link: origin xyz= -0.1 0 0 -> xyz= 0 0 0

Commit message: feat(ros2): update robot simulation setup and add SLAM assets
- Refine rover URDF configuration and Gazebo integration
- Update RViz visualization settings and remove obsolete displays
- Align spawn_robot launch arguments with package setup metadata
- Improve launch configuration consistency for simulation startup
- Add SLAM configuration and dedicated launch file
- Add saved SLAM map assets and serialized posegraph data

Updated:
- rover.urdf
- rover.rviz
- spawn_robot.launch.py
- setup.py

Added:
- slam.yaml
- slam.launch.py
- 21-05-2026.pgm
- 21-05-2026.yaml
- 21-05-2026.data
- 21-05-2026.posegraph

File: src/rover_description/urdf/rover.urdf (robot description, URDF)
Before this commit: robot rover_bot, 6 links, 5 joints
Links:
- added link chassis, mass 5.0; collision box size=0.5 0.3 0.1; visual box size=0.5 0.3 0.1
- link base_link: mass 5.0 -> None; geometry 
Joints:
- removed joint base_to_base_link
- added joint base_footprint_joint: type fixed, parent base_link, child base_footprint, origin xyz=0.0 0.0 0.0 rpy=0.0 0.0 0.0
- added joint base_to_chassis: type fixed, parent base_link, child chassis, origin xyz= 0 0 0
- joint caster_joint: parent base_link -> chassis
- joint left_wheel_joint: parent base_link -> chassis
- joint lidar_joint: parent base_link -> chassis
- joint right_wheel_joint: parent base_link -> chassis

Commit message: fix(urdf): correct robot frame hierarchy and align base_footprint with navigation stack
- Introduce proper separation between base_footprint (ground frame) and base_link (robot body center)
- Move base_footprint to ground level for accurate 2D navigation
- Attach base_link above base_footprint with vertical offset
- Fix chassis, wheel, and caster Z positions to match physical robot geometry
- Adjust LiDAR placement to ensure correct scan alignment with map
- Ensure consistent frame usage for DiffDrive, AMCL, and SLAM compatibility

File: src/rover_description/urdf/rover.urdf (robot description, URDF)
Before this commit: robot rover_bot, 7 links, 6 joints
Links:
- link lidar_link: geometry collision cylinder length=0.06 radius=0.05; visual cylinder length=0.06 radius=0.05
Joints:
- joint base_footprint_joint: child base_footprint -> base_link; origin xyz=0.0 0.0 0.0 rpy=0.0 0.0 0.0 -> xyz=0.0 0.0 0.07 rpy=0.0 0.0 0.0; parent base_link -> base_footprint
- joint caster_joint: origin xyz=-0.2 0 0.05 -> xyz=-0.2 0 -0.02
- joint left_wheel_joint: origin xyz=0.2 0.16 0.07 rpy=-1.57 0 0 -> xyz=0.2 0.16 0 rpy=-1.57 0 0
- joint lidar_joint: origin xyz=0.2 0 0.15 -> xyz=0.2 0 0.08
- joint right_wheel_joint: origin xyz=0.2 -0.16 0.07 rpy=1.57 0 0 -> xyz=0.2 -0.16 0 rpy=1.57 0 0
