Commit message: feat(sim): add camera sensor link, Gazebo configs, and gz-ROS bridge

File: src/diffbot_description/urdf/gazebo.xacro (robot description, xacro)
@@ -122,5 +122,5 @@
     </gazebo> -->
     <!-- Joint State Publisher -->
-    <gazebo>
+    <!-- <gazebo>
         <plugin filename="gz-sim-joint-state-publisher-system"
             name="gz::sim::systems::JointStatePublisher">
@@ -129,4 +129,26 @@
             <joint_name>right_wheel_joint</joint_name>
         </plugin>
+    </gazebo> -->
+    <!-- Camera Sensor configs -->
+    <gazebo reference="camera_link">
+        <sensor name="camera_sensor" type="camera">
+            <always_on>true</always_on>
+            <visualize>true</visualize>
+            <update_rate>30</update_rate>
+            <topic>/camera/image_raw</topic>
+            <camera>
+                <horizontal_fov>1.57</horizontal_fov>
+                <image>
+                    <width>640</width>
+                    <height>480</height>
+                    <format>R8G8B8</format>
+                </image>
+                <clip>
+                    <near>0.05</near>
+                    <far>20.0</far>
+                </clip>
+            </camera>
+            <gz_frame_id>camera_link</gz_frame_id>
+        </sensor>
     </gazebo>
     <!-- Plugins for Sensors -->

File: src/diffbot_description/urdf/materials.xacro (robot description, xacro)
@@ -7,3 +7,6 @@
         <color rgba="1 0 0 1"/>
     </material>
+    <material name="blue">
+        <color rgba="0 0.5 1 1"/>
+    </material>
 </robot>

File: src/diffbot_description/urdf/sensors.xacro (robot description, xacro)
@@ -31,4 +31,5 @@
         <origin xyz="0.2 0 0.08"/>
     </joint>
+    <!-- IMU -->
     <link name="imu_link">
         <visual>
@@ -59,3 +60,32 @@
         <origin xyz="0 0 0.06"/>
     </joint>
+    <!-- Camera -->
+    <link name="camera_link">
+        <visual>
+            <geometry>
+                <box size="0.02 0.02 0.02"/>
+            </geometry>
+            <material name="blue"/>
+        </visual>
+        <collision>
+            <geometry>
+                <box size="0.02 0.02 0.02"/>
+            </geometry>
+        </collision>
+        <inertial>
+            <mass value="0.01" />
+            <inertia
+                ixx="0.0001"
+                ixy="0"
+                ixz="0"
+                iyy="0.0001"
+                iyz="0"
+                izz="0.0001"/>
+        </inertial>
+    </link>
+    <joint name="camera_joint" type="fixed">
+        <parent link="chassis"/>
+        <child link="camera_link"/>
+        <origin xyz="0.25 0 0"/>
+    </joint>
 </robot>
